File: bk_amplifier_v0/bk_amplifier.sch (KiCad schematic (older format))
At the start: 8 parts, among them J1 Conn_Coaxial, J2 Conn_Coaxial, U1 AD745

Commit message: 1st components dimensionment
Parts:
- added R3: 470, symbol Device:R
- C1: value 370p -> 33p
- J2: Spice_Model 10k -> 100k
Connections:
- net GND: now also R3.2; no longer U1.3 (-)
- net Vcc: now also U1.13 (V+); no longer U1.6 (V-)
- net Vee: now also U1.6 (V-); no longer U1.13 (V+)
- net retro: now also U1.3 (-); no longer U1.5 (+)
- new net: R3.1, U1.5 (+)
Other:
- note added: "R3 = R2 to minimize offset error\ndue to input bias current"
- note added: "Voltage gain is given by Chydro/C1\nCharge gain is given by 1/C1, in Coulomb per Volt\nC1 should be in polystyren"
- note added: "high freq given by 1/2*pi*R2*Chydro"
- note removed: "gain is given by Cin/C1\nC1 in polystyren"
- note removed: "high freq given by 1/2*pi*R2*Cin"
Changed lines of the file:
@@
 U 1 1 5DA0556F
 P 5300 4550
-F 0 "R2" V 5093 4550 50  0000 C CNN
-F 1 "470" V 5184 4550 50  0000 C CNN
+F 0 "R2" V 5500 4500 50  0000 L BNN
+F 1 "470" V 5400 4500 50  0000 L BNN
 F 2 "" V 5230 4550 50  0001 C CNN
 F 3 "~" H 5300 4550 50  0001 C CNN
@@
 P 6500 3550
 F 0 "C1" V 6750 3550 50  0000 C CNN
-F 1 "370p" V 6650 3550 50  0000 C CNN
+F 1 "33p" V 6650 3550 50  0000 C CNN
 F 2 "" H 6538 3400 50  0001 C CNN
 F 3 "~" H 6500 3550 50  0001 C CNN
@@
 	-1   0    0    -1
 $EndComp
-Text Notes 6650 3500 0    50   ~ 0
-gain is given by Cin/C1\nC1 in polystyren
+Text Notes 5900 3150 0    50   ~ 0
+Voltage gain is given by Chydro/C1\nCharge gain is given by 1/C1, in Coulomb per Volt\nC1 should be in polystyren
 Text Notes 5950 3800 0    50   ~ 0
 low freq given by 1/2*pi*R1*C1
-Text Notes 4450 4350 0    50   ~ 0
-high freq given by 1/2*pi*R2*Cin
+Text Notes 4500 4250 0    50   ~ 0
+high freq given by 1/2*pi*R2*Chydro
 $Comp
 L pspice:VSOURCE V1
@@
 	5300 3200 5300 3250
 Wire Wire Line
-	4650 4750 6150 4750
-Wire Wire Line
 	5950 4550 6150 4550
 Connection ~ 5950 4550
@@
 Wire Wire Line
 	4850 4550 5000 4550
-Connection ~ 4650 4750
 $Comp
 L Connector:Conn_Coaxial J2
@@
 F 3 " ~" H 7500 4650 50  0001 C CNN
 F 4 "R" H 7500 4650 50  0001 C CNN "Spice_Primitive"
-F 5 "10k" H 7500 4650 50  0001 C CNN "Spice_Model"
+F 5 "100k" H 7500 4650 50  0001 C CNN "Spice_Model"
 F 6 "Y" H 7500 4650 50  0001 C CNN "Spice_Netlist_Enabled"
 	1    7500 4650
@@
 F 8 "5 3 13 6 12" H 6794 4559 50  0001 L CNN "Spice_Node_Sequence"
 	1    6450 4650
-	1    0    0    -1
-$EndComp
-Text Notes 5450 5050 0    50   ~ 0
+	1    0    0    1
+$EndComp
+Text Notes 6050 6050 0    50   ~ 0
 REF: SLOA033a
+$Comp
+L Device:R R3
+U 1 1 5DA73A7D
+P 5300 4750
+F 0 "R3" V 5500 4750 50  0000 C CNN
+F 1 "470" V 5400 4750 50  0000 C CNN
+F 2 "" V 5230 4750 50  0001 C CNN
+F 3 "~" H 5300 4750 50  0001 C CNN
+	1    5300 4750
+	0    1    1    0
+$EndComp
+Wire Wire Line
+	5450 4750 6150 4750
+Wire Wire Line
+	5150 4750 4650 4750
+Connection ~ 4650 4750
+Text Notes 4800 5200 0    50   ~ 0
+R3 = R2 to minimize offset error\ndue to input bias current
 $EndSCHEMATC
