File: bk_amplifier_v0/bk_amplifier.sch (KiCad schematic (older format))
At the start: 9 parts, among them J1 Conn_Coaxial, J2 Conn_Coaxial, U1 AD745

Commit message: a simulation bench for OpAmp
Parts:
- J1: Spice_Model BK8103_V -> BK8103_x
Connections:
- net pos: now reaches R3.1, U1.5 (+)
- net in renamed hydro
- net retro renamed neg
Other:
- note added: ".tran 1n 1m"
Changed lines of the file:
@@
 out
 Text GLabel 4850 4400 0    50   Input ~ 0
-in
-Text GLabel 5850 3550 0    50   BiDi ~ 0
-retro
-Wire Wire Line
-	5850 3550 5950 3550
-Connection ~ 5950 3550
+hydro
+Text GLabel 5950 4550 3    50   Input ~ 0
+neg
 Wire Wire Line
 	4850 4400 5000 4400
@@
 F 3 "doc/BK810x.pdf" H 4650 4550 50  0001 C CNN
 F 4 "X" H 4650 4550 50  0001 C CNN "Spice_Primitive"
-F 5 "BK8103_V" H 4650 4550 50  0001 C CNN "Spice_Model"
+F 5 "BK8103_x" H 4650 4550 50  0001 C CNN "Spice_Model"
 F 6 "Y" H 4650 4550 50  0001 C CNN "Spice_Netlist_Enabled"
 F 7 "bk8103.cir" H 4650 4550 50  0001 C CNN "Spice_Lib_File"
@@
 Text Notes 4800 5200 0    50   ~ 0
 R3 = R2 to minimize offset error\ndue to input bias current
+Text GLabel 5950 4750 3    50   Input ~ 0
+pos
+Text Notes 6700 5000 0    50   ~ 0
+.tran 1n 1m
 $EndSCHEMATC
